File: A4092.kicad_pcb (KiCad board)
At the start: 2 copper layers, 0 parts

Commit message: Finished first pass at new schematics
Parts:
- added C1: 100nF, Capacitor_SMD:C_0603_1608Metric_Pad1.08x0.95mm_HandSolder, F.Cu at (120.2, 100.1)
- added C10: 100pF, CA0612KRNPO9BN101:CAP_CA0612_3P2X1P6_YAG, F.Cu at (203.1, 88.3)
- added C11: 100nF, Capacitor_SMD:C_0603_1608Metric_Pad1.08x0.95mm_HandSolder, F.Cu at (190.2, 105.0)
- added C12: 100nF, Capacitor_SMD:C_0603_1608Metric_Pad1.08x0.95mm_HandSolder, F.Cu at (190.2, 107.5)
- added C13: 100nF, Capacitor_SMD:C_0603_1608Metric_Pad1.08x0.95mm_HandSolder, F.Cu at (190.2, 110.0)
- added C14: 100nF, Capacitor_SMD:C_0603_1608Metric_Pad1.08x0.95mm_HandSolder, F.Cu at (190.2, 112.5)
- added C15: 100nF, Capacitor_SMD:C_0603_1608Metric_Pad1.08x0.95mm_HandSolder, F.Cu at (190.2, 115.0)
- added C16: 100nF, Capacitor_SMD:C_0603_1608Metric_Pad1.08x0.95mm_HandSolder, F.Cu at (190.2, 117.5)
- added C17: 100nF, Capacitor_SMD:C_0603_1608Metric_Pad1.08x0.95mm_HandSolder, F.Cu at (190.2, 120.0)
- added C18: 100nF, Capacitor_SMD:C_0603_1608Metric_Pad1.08x0.95mm_HandSolder, F.Cu at (169.6, 129.7)
- added C19: 100nF, Capacitor_SMD:C_0603_1608Metric_Pad1.08x0.95mm_HandSolder, F.Cu at (169.6, 132.2)
- added C2: 4.7uF, Capacitor_SMD:CP_Elec_4x5.7, F.Cu at (103.2, 101.7)
- added C20: 100nF, Capacitor_SMD:C_0603_1608Metric_Pad1.08x0.95mm_HandSolder, F.Cu at (169.6, 134.8)
- added C21: 100nF, Capacitor_SMD:C_0603_1608Metric_Pad1.08x0.95mm_HandSolder, F.Cu at (169.6, 137.3)
- added C22: 100nF, Capacitor_SMD:C_0603_1608Metric_Pad1.08x0.95mm_HandSolder, F.Cu at (169.6, 139.8)
- added C23: 100nF, Capacitor_SMD:C_0603_1608Metric_Pad1.08x0.95mm_HandSolder, F.Cu at (173.9, 129.7)
- added C24: 100nF, Capacitor_SMD:C_0603_1608Metric_Pad1.08x0.95mm_HandSolder, F.Cu at (173.9, 132.2)
- added C25: 100nF, Capacitor_SMD:C_0603_1608Metric_Pad1.08x0.95mm_HandSolder, F.Cu at (173.9, 134.8)
- added C26: 100nF, Capacitor_SMD:C_0603_1608Metric_Pad1.08x0.95mm_HandSolder, F.Cu at (173.9, 137.3)
- added C27: 100nF, Capacitor_SMD:C_0603_1608Metric_Pad1.08x0.95mm_HandSolder, F.Cu at (173.9, 139.8)
- added C28: 100nF, Capacitor_SMD:C_0603_1608Metric_Pad1.08x0.95mm_HandSolder, F.Cu at (178.3, 129.7)
- added C29: 0.1uF, Capacitor_SMD:C_0603_1608Metric_Pad1.08x0.95mm_HandSolder, F.Cu at (178.3, 132.2)
- added C3: 100nF, Capacitor_SMD:C_0603_1608Metric_Pad1.08x0.95mm_HandSolder, F.Cu at (120.2, 102.6)
- added C30: 100nF, Capacitor_SMD:C_0603_1608Metric_Pad1.08x0.95mm_HandSolder, F.Cu at (178.3, 134.8)
- added C31: 100nF, Capacitor_SMD:C_0603_1608Metric_Pad1.08x0.95mm_HandSolder, F.Cu at (178.3, 137.3)
- added C32: 10nF, Capacitor_SMD:C_0603_1608Metric_Pad1.08x0.95mm_HandSolder, F.Cu at (173.0, 107.7)
- added C33: 47uF, Capacitor_SMD:CP_Elec_6.3x7.7, F.Cu at (136.1, 82.2)
- added C34: 100nF, Capacitor_SMD:C_0603_1608Metric_Pad1.08x0.95mm_HandSolder, F.Cu at (173.0, 110.2)
- added C35: 10nF, Capacitor_SMD:C_0603_1608Metric_Pad1.08x0.95mm_HandSolder, F.Cu at (173.0, 112.7)
- added C36: 100nF, Capacitor_SMD:C_0603_1608Metric_Pad1.08x0.95mm_HandSolder, F.Cu at (173.0, 115.2)
- added C37: 10nF, Capacitor_SMD:C_0603_1608Metric_Pad1.08x0.95mm_HandSolder, F.Cu at (173.0, 117.7)
- added C38: 100nF, Capacitor_SMD:C_0603_1608Metric_Pad1.08x0.95mm_HandSolder, F.Cu at (177.4, 107.7)
- added C39: 10nF, Capacitor_SMD:C_0603_1608Metric_Pad1.08x0.95mm_HandSolder, F.Cu at (177.4, 110.2)
- added C4: 4.7uF, Capacitor_SMD:CP_Elec_4x5.7, F.Cu at (103.2, 107.6)
- added C40: 100nF, Capacitor_SMD:C_0603_1608Metric_Pad1.08x0.95mm_HandSolder, F.Cu at (177.4, 112.7)
- added C41: 10nF, Capacitor_SMD:C_0603_1608Metric_Pad1.08x0.95mm_HandSolder, F.Cu at (177.4, 115.2)
- added C42: 100nF, Capacitor_SMD:C_0603_1608Metric_Pad1.08x0.95mm_HandSolder, F.Cu at (177.4, 117.7)
- added C43: 47uF, Capacitor_SMD:CP_Elec_6.3x7.7, F.Cu at (136.1, 90.3)
- added C44: 47uF, Capacitor_SMD:CP_Elec_6.3x7.7, F.Cu at (136.1, 98.5)
- added C45: 47uF, Capacitor_SMD:CP_Elec_6.3x7.7, F.Cu at (136.1, 106.6)
- added C5: 10pF, Capacitor_SMD:C_0603_1608Metric_Pad1.08x0.95mm_HandSolder, F.Cu at (185.4, 36.8)
- added C6: 100pF, CA0612KRNPO9BN101:CAP_CA0612_3P2X1P6_YAG, F.Cu at (185.8, 88.3)
- added C7: 100pF, CA0612KRNPO9BN101:CAP_CA0612_3P2X1P6_YAG, F.Cu at (190.2, 88.3)
- added C8: 100pF, CA0612KRNPO9BN101:CAP_CA0612_3P2X1P6_YAG, F.Cu at (194.5, 88.3)
- added C9: 100pF, CA0612KRNPO9BN101:CAP_CA0612_3P2X1P6_YAG, F.Cu at (198.8, 88.3)
- added CN1: Zorro3, Zorro3:Zorro3-CardEdge, F.Cu at (62.5, 152.3)
- added D1: SS24, Diode_SMD:D_SMA_Handsoldering, F.Cu at (199.4, 105.0)
- added F1: ASMDC185F/33-2, Fuse:Fuse_2920_7451Metric_Pad2.10x5.45mm_HandSolder, F.Cu at (200.7, 97.4)
- added FB1: 60, Capacitor_SMD:C_0603_1608Metric_Pad1.08x0.95mm_HandSolder, F.Cu at (181.7, 107.7)
- added FB2: 60, Capacitor_SMD:C_0603_1608Metric_Pad1.08x0.95mm_HandSolder, F.Cu at (181.7, 110.2)
- added FB3: 60, Capacitor_SMD:C_0603_1608Metric_Pad1.08x0.95mm_HandSolder, F.Cu at (181.7, 112.7)
- added FB4: 60, Capacitor_SMD:C_0603_1608Metric_Pad1.08x0.95mm_HandSolder, F.Cu at (185.4, 39.3)
- added FB5: 60, Capacitor_SMD:C_0603_1608Metric_Pad1.08x0.95mm_HandSolder, F.Cu at (185.4, 41.8)
- added FL1: DA1206D600R-10, DA1206D600R-10:FB_DA1206D600R-10, F.Cu at (187.5, 77.3)
- added FL10: DA1206D600R-10, DA1206D600R-10:FB_DA1206D600R-10, F.Cu at (205.4, 82.0)
- added FL2: DA1206D600R-10, DA1206D600R-10:FB_DA1206D600R-10, F.Cu at (192.0, 77.3)
- added FL3: DA1206D600R-10, DA1206D600R-10:FB_DA1206D600R-10, F.Cu at (196.5, 77.3)
- added FL4: DA1206D600R-10, DA1206D600R-10:FB_DA1206D600R-10, F.Cu at (200.9, 77.3)
- added FL5: DA1206D600R-10, DA1206D600R-10:FB_DA1206D600R-10, F.Cu at (205.4, 77.3)
- added FL6: DA1206D600R-10, DA1206D600R-10:FB_DA1206D600R-10, F.Cu at (187.5, 82.0)
- added FL7: DA1206D600R-10, DA1206D600R-10:FB_DA1206D600R-10, F.Cu at (192.0, 82.0)
- added FL8: DA1206D600R-10, DA1206D600R-10:FB_DA1206D600R-10, F.Cu at (196.5, 82.0)
- added FL9: DA1206D600R-10, DA1206D600R-10:FB_DA1206D600R-10, F.Cu at (200.9, 82.0)
- added J1: Conn_02x25_Odd_Even, Connector_IDC:IDC-Header_2x25_P2.54mm_Vertical, F.Cu at (109.8, 49.9)
- added J2: Conn_01x06_Pin, Connector_PinHeader_2.54mm:PinHeader_1x06_P2.54mm_Vertical, F.Cu at (65.8, 72.0)
- added J3: TO-LED, Connector_PinHeader_2.54mm:PinHeader_1x03_P2.54mm_Vertical, F.Cu at (64.8, 59.8)
- added J4: TO-MB, Connector_PinHeader_2.54mm:PinHeader_1x03_P2.54mm_Vertical, F.Cu at (77.8, 59.8)
- added J5: 5787170-5, 5787170_5:CONN_5787170-5_TYC, F.Cu at (217.9, 77.8)
- added J6: 350543-1, 350543_1:CONN_350543-1_TYC, F.Cu at (189.0, 127.6)
- added J7: 22112042, 22112042:CONN_A-6373-04A_MOL, F.Cu at (200.4, 135.9)
- added R1: 22, Resistor_SMD:R_0603_1608Metric_Pad0.98x0.95mm_HandSolder, F.Cu at (181.7, 115.2)
- added R10: 1K, YC324-FK-071KL:RESCAXS127P508X320X70-8N, F.Cu at (170.6, 100.0)
- added R11: 120, Resistor_SMD:R_0603_1608Metric, F.Cu at (185.9, 110.2)
- added R12: 1K, YC324-FK-071KL:RESCAXS127P508X320X70-8N, F.Cu at (39.4, 109.2)
- added R13: 1K, YC324-FK-071KL:RESCAXS127P508X320X70-8N, F.Cu at (45.9, 109.2)
- added R14: 1K, YC324-FK-071KL:RESCAXS127P508X320X70-8N, F.Cu at (52.4, 109.2)
- added R15: 1K, YC324-FK-071KL:RESCAXS127P508X320X70-8N, F.Cu at (58.9, 109.2)
- added R16: 1K, YC324-FK-071KL:RESCAXS127P508X320X70-8N, F.Cu at (65.5, 109.2)
- added R17: 1K, YC324-FK-071KL:RESCAXS127P508X320X70-8N, F.Cu at (177.1, 100.0)
- added R2: 22, Resistor_SMD:R_0603_1608Metric_Pad0.98x0.95mm_HandSolder, F.Cu at (181.7, 117.7)
- added R4: YC324-FK-071KL, YC324-FK-071KL:RESCAXS127P508X320X70-8N, F.Cu at (102.9, 95.5)
- added R5: YC324-FK-071KL, YC324-FK-071KL:RESCAXS127P508X320X70-8N, F.Cu at (109.5, 95.5)
- added R6: 1K, YC324-FK-071KL:RESCAXS127P508X320X70-8N, F.Cu at (151.0, 100.0)
- added R7: 1K, YC324-FK-071KL:RESCAXS127P508X320X70-8N, F.Cu at (157.5, 100.0)
- added R8: 1K, YC324-FK-071KL:RESCAXS127P508X320X70-8N, F.Cu at (164.1, 100.0)
- added R9: 120, Resistor_SMD:R_0603_1608Metric, F.Cu at (185.9, 107.7)
- added SW1: 219-8MST, 219_8MST:SO16_219-8_CTS, F.Cu at (215.7, 136.2)
- added U1: CY74FCT16543TPVCT, 74FCT16543:DL56, F.Cu at (135.2, 133.8)
- added U10: SN74F244DB, SN74F244DB:DB20, F.Cu at (112.7, 110.2)
- added U11: SN74ABT16374ADGGR, SN74ABT16374ADGGR:DGG48, F.Cu at (60.0, 132.3)
- added U12: 74LVC07APW_118, 74LVC07APW_118:TSSOP14_5P1X4P5_NEX, F.Cu at (81.0, 128.5)
- added U13: SN74ABT16245ADGGR, SN74ABT16245ADGGR:DGG48, F.Cu at (71.0, 132.3)
- added U14: 74ACT521MTCX, 74ACT521MTCX:TSSOP20_4P4X6P5_ONS, F.Cu at (81.1, 136.0)
- added U15: 74ABT74, Package_SO:TSSOP-14_4.4x5mm_P0.65mm, F.Cu at (164.8, 119.5)
- added U2: CY74FCT16543TPVCT, 74FCT16543:DL56, F.Cu at (103.9, 133.8)
- added U3: CY74FCT16543TPVCT, 74FCT16543:DL56, F.Cu at (120.0, 133.8)
- added U4: NCR53c710 SCSI Host Controller, Package_QFP:PQFP-160_28x28mm_P0.65mm, F.Cu at (164.6, 76.4)
- added U5: CY74FCT543ATQCT, 74FCT16543:DL56, F.Cu at (150.6, 134.0)
- added U6: ATF1508AS-10AU100, ATF1508AS:100A_ATM, F.Cu at (71.2, 88.8)
- added U7: SST39SF010, Package_SO:TSSOP-32_8x11mm_P0.65mm, F.Cu at (97.3, 78.2)
- added U8: DS21S07A, Package_SO:TSSOP-20_4.4x6.5mm_P0.65mm, F.Cu at (199.1, 58.7)
- added U9: DS21S07A, Package_SO:TSSOP-20_4.4x6.5mm_P0.65mm, F.Cu at (199.1, 66.8)
- added Y1: Abracon ACO-50MHz, Oscillator:Oscillator_DIP-14, F.Cu at (75.1, 113.2)
Other:
- board outline added: 192.7 x 123.3 mm
