File: zorro3.kicad_sch (KiCad schematic)
At the start: 17 parts, among them CN1 Zorro3, U1 SN74ABT16543DGGR, U11 SN74ABT16374ADGGR, U12 74LVC07APW_118, U13 SN74ABT16245ADGGR, U14 74ACT521MTCX, U2 SN74ABT16543DGGR, U3 SN74ABT16543DGGR, U5 CY74FCT543ATQCT

Commit message: Move to XC95144XL
and other changes related to that.
Parts:
- removed RN12, RN13: 1K, CAY16_102J4LF:BO_CAY16, symbol YC324-FK-071KL:YC324-FK-071KL
- removed U11: SN74ABT16374ADGGR, SN74ABT16374ADGGR:DGG48, symbol SN74ABT16374ADGGR:SN74ABT16374ADGGR
- removed U14: 74ACT521MTCX, 74ACT521MTCX:TSSOP20_4P4X6P5_ONS, symbol 74ACT521MTCX:74ACT521MTCX
- removed U5: CY74FCT543ATQCT, CY74FCT543ATQCT:DBQ24, symbol CY74FCT543ATQCT:CY74FCT543ATQCT
- added U6: SN74ABT16543DGGR, 74FCT16543:DL56, symbol 74FCT16543:CY74FCT16543TPVCT
Connections:
- net A10: now also U6.12 (1A6)
- net A11: now also U6.10 (1A5)
- net A12: now also U6.9 (1A4)
- net A13: now also U6.8 (1A3)
- net A14: now also U6.6 (1A2)
- net A15: now also U6.5 (1A1)
- net A8: now also U6.14 (1A8)
- net A9: now also U6.13 (1A7)
- net ABOEH: now also U6.56 (*1OEBA)
- net BMASTER: now also U6.54 (*1CEBA)
- net GND: now also U6.11 (GND), U6.18 (GND), U6.2 (*1LEAB), U6.25 (GND), U6.26 (*2CEAB), U6.27 (*2LEAB), U6.28 (*2OEAB), U6.29 (*2OEBA), U6.30 (*2LEBA), U6.31 (*2CEBA), U6.32 (GND), U6.39 (GND), U6.4 (GND), U6.46 (GND), U6.53 (GND)
- net IORST: now also U6.1 (*1OEAB)
- net MASTER: now also U6.3 (*1CEAB)
- net PLD_FCS: now also U6.55 (*1LEBA)
- net V5: now also U6.22 (VCC), U6.35 (VCC), U6.50 (VCC), U6.7 (VCC)
- net Z_A10D2: now also U6.45 (1B6)
- net Z_A11D3: now also U6.47 (1B5)
- net Z_A12D4: now also U6.48 (1B4)
- net Z_A13D5: now also U6.49 (1B3)
- net Z_A14D6: now also U6.51 (1B2)
- net Z_A15D7: now also U6.52 (1B1)
- net Z_A8D0: now also U6.43 (1B8)
- net Z_A9D1: now also U6.44 (1B7)
- no-connect marks 22 -> 37
Other:
- note removed: "2x8bit register w/ 3state"
- note removed: "Identity Comparator"
- note removed: "TODO 1x374 + 521 move into CPLD"
- note removed: "U100 / U101"
- note removed: "U107 / U106"
- note removed: "U108 / U105"
- moved on the sheet: CN1B, FB4, FB5, RN14, RN15, RN16, U12, U13, U3
