File: Kicad/Studies/A4092_0418.kicad_pcb (KiCad board)
At the start: 4 copper layers, 175.6 x 122.1 mm, 106 parts, among them CN1 Zorro3, J1 Conn_02x25_Odd_Even, J2 Conn_01x06_Pin, J3 TO-LED, J4 TO-MB, J5 5787170-5, J7 22112042, J8 TO-A3000-LED, J9 TO-A3000-MB, SW1 219-8MST, U1 SN74ABT16543DGGR, U10 NCR53c710 SCSI Host Controller, U11 DS21S07A, U12 DS21S07A, U13 SST39SF010, U2 SN74ABT16543DGGR, U3 SN74ABT16543DGGR, U4 SN74ABT16543DGGR, U5 74LVC07APW_118, U6 SN74ABT16245ADGGR, U7 AMS1117-3.3, U8 SN74F244DB, U9 XC95144XL-TQ144, Y1 Abracon ACO-50MHz

Commit message: routing progress
Parts:
- moved FB6 21.8 mm to (100.0, 92.0), turned to 180 degrees
- moved FB8 21.3 mm to (93.5, 102.0)
- moved FB7 21.0 mm to (90.0, 102.0)
- turned U9 to -90 degrees
Routing:
- net Z_INT2: track 76.4 -> 0.00 mm
- net A26: track 101.6 -> 35.3 mm, vias 3 -> 1
- net A25: track 102.4 -> 36.8 mm, vias 3 -> 1
- net A27: track 100.4 -> 36.8 mm, vias 3 -> 1
- net Z2D: track 60.1 -> 0.00 mm
- net BMASTER: track 58.8 -> 0.00 mm
- net D2Z: track 56.1 -> 0.00 mm
- net ABOEH: track 50.8 -> 0.00 mm
- net A28: track 94.8 -> 45.6 mm, vias 3 -> 1
- net DBOE: track 46.4 -> 0.00 mm
- net A24: track 63.8 -> 17.8 mm, vias 3 -> 1
- net DBLT: track 45.4 -> 0.00 mm
- net A30: track 89.1 -> 44.8 mm, vias 3 -> 1
- net A29: track 93.0 -> 48.8 mm, vias 3 -> 1
- net PLD_DS3: track 13.9 -> 57.9 mm, vias 1 -> 0
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