File: Kicad/A4092/scsi2.kicad_sch (KiCad schematic)
At the start: 28 parts, among them J3 TO-LED, J4 TO-MB, J8 TO-A3000-LED, J9 TO-A3000-MB, U10 NCR53c710 SCSI Host Controller, Y1 Abracon ACO-50MHz

Commit message: Update JLCPCB part numbers
Move to available and, if possible, basic parts
Parts:
- C1002, C1004, C1006, C1008, C32: LCSC Part # C100042 -> C57112
- R10: LCSC Part # C114662 -> C4190
- R11: LCSC Part # C95177 -> C23345
- R9: LCSC Part # C114640 -> C22787
Changed lines of the file:
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@@
 			)
 		)
-		(property "LCSC Part #" "C100042"
+		(property "LCSC Part #" "C57112"
 			(at 231.14 129.54 0)
 			(effects
@@
 			)
 		)
-		(property "LCSC Part #" "C95177"
+		(property "LCSC Part #" "C23345"
 			(at 259.08 130.81 90)
 			(effects
@@
 			)
 		)
-		(property "LCSC Part #" "C100042"
+		(property "LCSC Part #" "C57112"
 			(at 165.1 46.99 0)
 			(effects
@@
 			)
 		)
-		(property "LCSC Part #" "C100042"
+		(property "LCSC Part #" "C57112"
 			(at 182.88 67.31 0)
 			(effects
@@
 			)
 		)
-		(property "LCSC Part #" "C114640"
+		(property "LCSC Part #" "C22787"
 			(at 189.23 137.16 90)
 			(effects
@@
 			)
 		)
-		(property "LCSC Part #" "C100042"
+		(property "LCSC Part #" "C57112"
 			(at 199.39 46.99 0)
 			(effects
@@
 			)
 		)
-		(property "LCSC Part #" "C114662"
+		(property "LCSC Part #" "C4190"
 			(at 193.04 148.59 90)
 			(effects
@@
 			)
 		)
-		(property "LCSC Part #" "C100042"
+		(property "LCSC Part #" "C57112"
 			(at 182.88 26.67 0)
 			(effects
