File: Kicad/A4092/scsi2.kicad_sch (KiCad schematic)
At the start: 28 parts, among them J3 TO-LED, J4 TO-MB, J8 TO-A3000-LED, J9 TO-A3000-MB, U10 NCR53c710 SCSI Host Controller, Y1 Abracon ACO-50MHz

Commit message: Add rotations for all parts
Parts:
- J3, J4, J8, J9, RN10, RN17, RN6, RN7, RN8: FT Rotation Offset (none) -> 90
- Y1: FT Rotation Offset (none) -> 270
Changed lines of the file:
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@@
+			)
+		)
+		(property "FT Rotation Offset" "90"
+			(at 129.54 102.87 90)
+			(effects
+				(font
+					(size 1.27 1.27)
+				)
+				(hide yes)
 			)
 		)
@@
 			)
 		)
+		(property "FT Rotation Offset" "90"
+			(at 148.59 138.43 90)
+			(effects
+				(font
+					(size 1.27 1.27)
+				)
+				(hide yes)
+			)
+		)
 		(pin "1"
 		)
@@
 			)
 		)
+		(property "FT Rotation Offset" "90"
+			(at 148.59 102.87 90)
+			(effects
+				(font
+					(size 1.27 1.27)
+				)
+				(hide yes)
+			)
+		)
 		(pin "8"
 		)
@@
 		)
 		(property "LCSC Part #" "C7431196"
+			(at 248.92 130.81 0)
+			(effects
+				(font
+					(size 1.27 1.27)
+				)
+				(hide yes)
+			)
+		)
+		(property "FT Rotation Offset" "270"
 			(at 248.92 130.81 0)
 			(effects
@@
 			)
 		)
+		(property "FT Rotation Offset" "90"
+			(at 129.54 138.43 90)
+			(effects
+				(font
+					(size 1.27 1.27)
+				)
+				(hide yes)
+			)
+		)
 		(pin "5"
 		)
@@
 			)
 		)
+		(property "FT Rotation Offset" "90"
+			(at 172.72 100.33 0)
+			(effects
+				(font
+					(size 1.27 1.27)
+				)
+				(hide yes)
+			)
+		)
 		(pin "1"
 		)
@@
 			)
 		)
+		(property "FT Rotation Offset" "90"
+			(at 129.54 172.72 90)
+			(effects
+				(font
+					(size 1.27 1.27)
+				)
+				(hide yes)
+			)
+		)
 		(pin "1"
 		)
@@
 			)
 		)
+		(property "FT Rotation Offset" "90"
+			(at 194.31 121.92 0)
+			(effects
+				(font
+					(size 1.27 1.27)
+				)
+				(hide yes)
+			)
+		)
 		(pin "2"
 		)
@@
 		)
 		(property "LCSC Part #" "C6332196"
+			(at 172.72 121.92 0)
+			(effects
+				(font
+					(size 1.27 1.27)
+				)
+				(hide yes)
+			)
+		)
+		(property "FT Rotation Offset" "90"
 			(at 172.72 121.92 0)
 			(effects
@@
 			(at 194.31 100.33 0)
 			(effects
+				(font
+					(size 1.27 1.27)
+				)
+				(hide yes)
+			)
+		)
+		(property "FT Rotation Offset" "90"
+			(at 194.31 100.33 0)
+			(effects
