File: Kicad/A4092/zorro3.kicad_sch (KiCad schematic)
At the start: 13 parts, among them CN1 Zorro3, U1 SN74ABT16543DGGR, U2 SN74ABT16543DGGR, U3 SN74ABT16543DGGR, U4 SN74ABT16543DGGR, U5 74LVC07APW_118, U6 SN74ABT16245ADGGR

Commit message: Update to use new footprint for U1,2,3,4
Parts:
- U1, U2, U3, U4: footprint 74FCT16543:DL56 -> DGG56; symbol 74FCT16543:CY74FCT16543TPVCT -> SN74ABT16543DGGR:SN74ABT16543DGGR
Changed lines of the file:
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@@
 	)
 	(symbol
-		(lib_id "74FCT16543:CY74FCT16543TPVCT")
+		(lib_name "SN74ABT16543DGGR_1")
+		(lib_id "SN74ABT16543DGGR:SN74ABT16543DGGR")
 		(at 125.73 118.11 0)
 		(unit 1)
@@
 			)
 		)
-		(property "Footprint" "74FCT16543:DL56"
+		(property "Footprint" "DGG56"
 			(at 125.73 118.11 0)
 			(effects
@@
 	)
 	(symbol
-		(lib_id "74FCT16543:CY74FCT16543TPVCT")
+		(lib_id "SN74ABT16543DGGR:SN74ABT16543DGGR")
 		(at 27.94 31.75 0)
 		(unit 1)
@@
 			)
 		)
-		(property "Footprint" "74FCT16543:DL56"
+		(property "Footprint" "DGG56"
 			(at 27.94 31.75 0)
 			(effects
@@
 	)
 	(symbol
-		(lib_id "74FCT16543:CY74FCT16543TPVCT")
+		(lib_name "SN74ABT16543DGGR_2")
+		(lib_id "SN74ABT16543DGGR:SN74ABT16543DGGR")
 		(at 27.94 118.11 0)
 		(unit 1)
@@
 			)
 		)
-		(property "Footprint" "74FCT16543:DL56"
+		(property "Footprint" "DGG56"
 			(at 27.94 118.11 0)
 			(effects
@@
 	)
 	(symbol
-		(lib_id "74FCT16543:CY74FCT16543TPVCT")
+		(lib_name "SN74ABT16543DGGR_3")
+		(lib_id "SN74ABT16543DGGR:SN74ABT16543DGGR")
 		(at 125.73 30.48 0)
 		(unit 1)
@@
 			)
 		)
-		(property "Footprint" "74FCT16543:DL56"
+		(property "Footprint" "DGG56"
 			(at 125.73 30.48 0)
 			(effects
