File: Kicad/A4092/zorro3.kicad_sch (KiCad schematic)
At the start: 13 parts, among them CN1 Zorro3, U1 SN74ABT16543DGGR, U2 SN74ABT16543DGGR, U3 SN74ABT16543DGGR, U4 SN74ABT16543DGGR, U5 74LVC07APW_118, U6 SN74ABT16245ADGGR

Commit message: Add rotations for all parts
Parts:
- RN14, RN15, RN16: FT Rotation Offset (none) -> 90
- U1, U2, U3, U4, U5, U6: FT Rotation Offset (none) -> 270
Changed lines of the file:
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@@
+			)
+		)
+		(property "FT Rotation Offset" "90"
+			(at 259.08 118.11 90)
+			(effects
+				(font
+					(size 1.27 1.27)
+				)
+				(hide yes)
 			)
 		)
@@
 		)
 		(property "LCSC Part #" "C784824"
+			(at 278.13 118.11 90)
+			(effects
+				(font
+					(size 1.27 1.27)
+				)
+				(hide yes)
+			)
+		)
+		(property "FT Rotation Offset" "90"
 			(at 278.13 118.11 90)
 			(effects
@@
 			)
 		)
+		(property "FT Rotation Offset" "270"
+			(at 125.73 118.11 0)
+			(effects
+				(font
+					(size 1.27 1.27)
+				)
+				(hide yes)
+			)
+		)
 		(pin "8"
 		)
@@
 		)
 		(property "LCSC Part #" "C2865087"
+			(at 27.94 31.75 0)
+			(effects
+				(font
+					(size 1.27 1.27)
+				)
+				(hide yes)
+			)
+		)
+		(property "FT Rotation Offset" "270"
 			(at 27.94 31.75 0)
 			(effects
@@
 			)
 		)
+		(property "FT Rotation Offset" "270"
+			(at 27.94 118.11 0)
+			(effects
+				(font
+					(size 1.27 1.27)
+				)
+				(hide yes)
+			)
+		)
 		(pin "44"
 		)
@@
 		)
 		(property "LCSC Part #" "C6051"
+			(at 44.45 215.9 0)
+			(effects
+				(font
+					(size 1.27 1.27)
+				)
+				(hide yes)
+			)
+		)
+		(property "FT Rotation Offset" "270"
 			(at 44.45 215.9 0)
 			(effects
@@
 			)
 		)
+		(property "FT Rotation Offset" "90"
+			(at 260.35 165.1 90)
+			(effects
+				(font
+					(size 1.27 1.27)
+				)
+				(hide yes)
+			)
+		)
 		(pin "1"
 		)
@@
 		)
 		(property "LCSC Part #" "C130197"
+			(at 236.22 31.75 0)
+			(effects
+				(font
+					(size 1.27 1.27)
+				)
+				(hide yes)
+			)
+		)
+		(property "FT Rotation Offset" "270"
 			(at 236.22 31.75 0)
 			(effects
@@
 			(at 125.73 30.48 0)
 			(effects
+				(font
+					(size 1.27 1.27)
+				)
+				(hide yes)
+			)
+		)
+		(property "FT Rotation Offset" "270"
+			(at 125.73 30.48 0)
+			(effects
