File: Kicad/A4092/Termination.kicad_sch (KiCad schematic)
At the start: 29 parts, among them J1 Conn_02x25_Odd_Even, J5 Conn_02x25_Odd_Even, SW1 219-8MST, U11 DS21S07A, U12 DS21S07A, U8 SN74F244DB

Commit message: Update JLCPCB part numbers
Move to available and, if possible, basic parts
Parts:
- R1: LCSC Part # C95177 -> C21189
- R2: LCSC Part # C99782 -> C23162
Changed lines of the file:
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@@
 			)
 		)
-		(property "LCSC Part #" "C99782"
+		(property "LCSC Part #" "C23162"
 			(at 88.9 151.13 90)
 			(effects
@@
 			)
 		)
-		(property "LCSC Part #" "C95177"
+		(property "LCSC Part #" "C21189"
 			(at 95.25 154.94 90)
 			(effects

Commit message: Fix up capacitor array footprint
家裡創 did not like the digikey footprint.
Parts:
- C10, C6, C7, C8, C9: footprint CA0612KRNPO9BN101:CAP_CA0612_3P2X1P6_YAG -> CA0612KRNPO9BN101:CAP_CA0612_3P2X1P6_YAG-S
Changed lines of the file:
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@@
 			)
 		)
-		(property "Footprint" "CA0612KRNPO9BN101:CAP_CA0612_3P2X1P6_YAG"
+		(property "Footprint" "CA0612KRNPO9BN101:CAP_CA0612_3P2X1P6_YAG-S"
 			(at 244.856 75.184 0)
 			(effects
@@
 			)
 		)
-		(property "Footprint" "CA0612KRNPO9BN101:CAP_CA0612_3P2X1P6_YAG"
+		(property "Footprint" "CA0612KRNPO9BN101:CAP_CA0612_3P2X1P6_YAG-S"
 			(at 242.316 115.316 0)
 			(effects
@@
 			)
 		)
-		(property "Footprint" "CA0612KRNPO9BN101:CAP_CA0612_3P2X1P6_YAG"
+		(property "Footprint" "CA0612KRNPO9BN101:CAP_CA0612_3P2X1P6_YAG-S"
 			(at 227.076 33.274 0)
 			(effects
@@
 			)
 		)
-		(property "Footprint" "CA0612KRNPO9BN101:CAP_CA0612_3P2X1P6_YAG"
+		(property "Footprint" "CA0612KRNPO9BN101:CAP_CA0612_3P2X1P6_YAG-S"
 			(at 239.776 33.274 0)
 			(effects
@@
 			)
 		)
-		(property "Footprint" "CA0612KRNPO9BN101:CAP_CA0612_3P2X1P6_YAG"
+		(property "Footprint" "CA0612KRNPO9BN101:CAP_CA0612_3P2X1P6_YAG-S"
 			(at 232.664 115.316 0)
 			(effects

Commit message: Add rotations for all parts
Parts:
- C10, C6, C7, C8, C9, FL1, FL10, FL2, FL3, FL4, FL5, FL6, FL7, FL8, FL9: FT Rotation Offset (none) -> 90
- C1102, C1202: FT Rotation Offset (none) -> 180
- J1, J5: FT Rotation Offset (none) -> 270
Changed lines of the file:
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@@
 			)
 		)
+		(property "FT Rotation Offset" "90"
+			(at 102.87 59.69 90)
+			(effects
+				(font
+					(size 1.27 1.27)
+				)
+				(hide yes)
+			)
+		)
 		(pin "1"
 		)
@@
 			)
 		)
+		(property "FT Rotation Offset" "90"
+			(at 201.93 83.82 90)
+			(effects
+				(font
+					(size 1.27 1.27)
+				)
+				(hide yes)
+			)
+		)
 		(pin "1"
 		)
@@
 			)
 		)
+		(property "FT Rotation Offset" "90"
+			(at 238.76 76.2 90)
+			(effects
+				(font
+					(size 1.27 1.27)
+				)
+				(hide yes)
+			)
+		)
 		(pin "8"
 		)
@@
 			)
 		)
+		(property "FT Rotation Offset" "90"
+			(at 201.93 106.68 90)
+			(effects
+				(font
+					(size 1.27 1.27)
+				)
+				(hide yes)
+			)
+		)
 		(pin "1"
 		)
@@
 			)
 		)
+		(property "FT Rotation Offset" "90"
+			(at 236.22 114.3 90)
+			(effects
+				(font
+					(size 1.27 1.27)
+				)
+				(hide yes)
+			)
+		)
 		(pin "7"
 		)
@@
 			)
 		)
+		(property "FT Rotation Offset" "90"
+			(at 201.93 120.65 90)
+			(effects
+				(font
+					(size 1.27 1.27)
+				)
+				(hide yes)
+			)
+		)
 		(pin "7"
 		)
@@
 			)
 		)
+		(property "FT Rotation Offset" "180"
+			(at 26.67 48.26 0)
+			(effects
+				(font
+					(size 1.27 1.27)
+				)
+				(hide yes)
+			)
+		)
 		(pin "1"
 		)
@@
 			)
 		)
+		(property "FT Rotation Offset" "180"
+			(at 26.67 82.55 0)
+			(effects
+				(font
+					(size 1.27 1.27)
+				)
+				(hide yes)
+			)
+		)
 		(pin "1"
 		)
@@
 			)
 		)
+		(property "FT Rotation Offset" "90"
+			(at 220.98 34.29 90)
+			(effects
+				(font
+					(size 1.27 1.27)
+				)
+				(hide yes)
+			)
+		)
 		(pin "2"
 		)
@@
 			)
 		)
+		(property "FT Rotation Offset" "90"
+			(at 140.97 59.69 90)
+			(effects
+				(font
+					(size 1.27 1.27)
+				)
+				(hide yes)
+			)
+		)
 		(pin "1"
 		)
@@
 			)
 		)
+		(property "FT Rotation Offset" "90"
+			(at 116.84 59.69 90)
+			(effects
+				(font
+					(size 1.27 1.27)
+				)
+				(hide yes)
+			)
+		)
 		(pin "7"
 		)
@@
 			)
 		)
+		(property "FT Rotation Offset" "90"
+			(at 233.68 34.29 90)
+			(effects
+				(font
+					(size 1.27 1.27)
+				)
+				(hide yes)
+			)
+		)
 		(pin "5"
 		)
@@
 			)
 		)
+		(property "FT Rotation Offset" "90"
+			(at 201.93 54.61 90)
+			(effects
+				(font
+					(size 1.27 1.27)
+				)
+				(hide yes)
+			)
+		)
 		(pin "1"
 		)
@@
 			)
 		)
+		(property "FT Rotation Offset" "90"
+			(at 168.91 59.69 90)
+			(effects
+				(font
+					(size 1.27 1.27)
+				)
+				(hide yes)
+			)
+		)
 		(pin "1"
 		)
@@
 			)
 		)
+		(property "FT Rotation Offset" "90"
+			(at 154.94 59.69 90)
+			(effects
+				(font
+					(size 1.27 1.27)
+				)
+				(hide yes)
+			)
+		)
 		(pin "7"
 		)
@@
 			)
 		)
+		(property "FT Rotation Offset" "270"
+			(at 266.7 77.47 90)
+			(effects
+				(font
+					(size 1.27 1.27)
+				)
+				(hide yes)
+			)
+		)
 		(pin "1"
 		)
@@
 			)
 		)
+		(property "FT Rotation Offset" "90"
+			(at 201.93 68.58 90)
+			(effects
+				(font
+					(size 1.27 1.27)
+				)
+				(hide yes)
+			)
+		)
 		(pin "7"
 		)
@@
 			)
 		)
+		(property "FT Rotation Offset" "90"
+			(at 238.76 114.3 90)
+			(effects
+				(font
+					(size 1.27 1.27)
+				)
+				(hide yes)
+			)
+		)
 		(pin "4"
 		)
@@
 			(at 121.92 34.29 90)
 			(effects
+				(font
+					(size 1.27 1.27)
+				)
+				(hide yes)
+			)
+		)
+		(property "FT Rotation Offset" "270"
+			(at 121.92 34.29 90)
+			(effects
