File: Kicad/A4092/cpld.kicad_sch (KiCad schematic)
At the start: 15 parts, among them J2 Conn_01x06_Pin, U7 AMS1117-3.3, U9 XC95144XL-TQ144

Commit message: Add rotations for all parts
Parts:
- C702: FT Rotation Offset (none) -> 180
- RN1: FT Rotation Offset (none) -> 90
Changed lines of the file:
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@@
+			)
+		)
+		(property "FT Rotation Offset" "180"
+			(at 168.91 97.79 0)
+			(effects
+				(font
+					(size 1.27 1.27)
+				)
+				(hide yes)
 			)
 		)
@@
 			(at 170.18 33.02 0)
 			(effects
+				(font
+					(size 1.27 1.27)
+				)
+				(hide yes)
+			)
+		)
+		(property "FT Rotation Offset" "90"
+			(at 170.18 33.02 0)
+			(effects
