File: Kicad/A4092/flash.kicad_sch (KiCad schematic)
At the start: 5 parts, among them U13 SST39SF010/020/040, U14 W25X40CLSN

Commit message: Update JLCPCB part numbers
Move to available and, if possible, basic parts
Parts:
- R1401: LCSC Part # C22548 -> C25804
- U13: LCSC Part # C630569 -> C72450
- U14: LCSC Part # (none) -> C19617
Changed lines of the file:
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@@
 			)
 		)
-		(property "LCSC Part #" "C630569"
+		(property "LCSC Part #" "C72450"
 			(at 63.5 66.04 0)
 			(effects
@@
 			)
 		)
+		(property "LCSC Part #" " C19617"
+			(at 124.46 46.99 0)
+			(effects
+				(font
+					(size 1.27 1.27)
+				)
+				(hide yes)
+			)
+		)
 		(pin "8"
 		)
@@
 			)
 		)
-		(property "LCSC Part #" "C22548"
+		(property "LCSC Part #" "C25804"
 			(at 109.22 35.56 0)
 			(effects

Commit message: Add rotations for all parts
Parts:
- U13: FT Rotation Offset (none) -> 270
Changed lines of the file:
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@@
+			)
+		)
+		(property "FT Rotation Offset" "270"
+			(at 63.5 66.04 0)
+			(effects
+				(font
+					(size 1.27 1.27)
+				)
+				(hide yes)
 			)
 		)
