File: Kicad/A4092/flash.kicad_sch (KiCad schematic)
At the start: 5 parts, among them U13 SST39SF010/020/040, U14 W25X40CLSN

Commit message: Remove spaces from JLCPCB part numbers
Parts:
- U14: LCSC Part # C19617 -> C19617
Changed lines of the file:
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@@
 			)
 		)
-		(property "LCSC Part #" " C19617"
+		(property "LCSC Part #" "C19617"
 			(at 124.46 46.99 0)
 			(effects
