File: Kicad/Terminator-LT1118-2.85/A4092-terminator.kicad_sch (KiCad schematic)
At the start: 10 parts, among them J1 Conn_02x25_Odd_Even, U1 LT1118-2.85

Commit message: Update LT1118-2.85 based terminator
Parts:
- R3: LCSC Part # (none) -> C25803
- RN1, RN2, RN3, RN4, RN5: LCSC Part # C176176 -> C474279
Changed lines of the file:
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@@
 			)
 		)
-		(property "LCSC Part #" "C176176"
+		(property "LCSC Part #" "C474279"
 			(at 135.89 39.37 0)
 			(effects
@@
 			)
 		)
-		(property "LCSC Part #" "C176176"
+		(property "LCSC Part #" "C474279"
 			(at 97.79 63.5 0)
 			(effects
@@
 			)
 		)
-		(property "LCSC Part #" "C176176"
+		(property "LCSC Part #" "C474279"
 			(at 135.89 63.5 0)
 			(effects
@@
 			)
 		)
-		(property "LCSC Part #" "C176176"
+		(property "LCSC Part #" "C474279"
 			(at 172.72 39.37 0)
 			(effects
@@
 			)
 		)
-		(property "LCSC Part #" "C176176"
+		(property "LCSC Part #" "C474279"
 			(at 97.79 39.37 0)
 			(effects
@@
 			)
 		)
-		(property "LCSC Part #" ""
+		(property "LCSC Part #" "C25803"
 			(at 165.1 58.42 90)
 			(effects
