File: Kicad/Terminator-dev/A4092-terminator-dev.kicad_sch (KiCad schematic)
At the start: 14 parts, among them J1 Conn_02x25_Odd_Even, Q1 AO3401A, U1 LT1118-2.85

Commit message: Update DEV version of the terminator
with switch for experimenting w/ mosfet
Parts:
- J1: footprint Connector_IDC:IDC-Header_2x25_P2.54mm_Horizontal -> Connector_IDC_local:IDC-Header_2x25_P2.54mm_Horizontal
Changed lines of the file:
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@@
 			)
 		)
-		(property "Footprint" "Connector_IDC:IDC-Header_2x25_P2.54mm_Horizontal"
+		(property "Footprint" "Connector_IDC_local:IDC-Header_2x25_P2.54mm_Horizontal"
 			(at 105.41 124.46 0)
 			(effects
